Commit message: DIFF: Some changes

File: cad/sigma.urdf (robot description, URDF)
Before this commit: robot sigma, 19 links, 18 joints
Links:
- removed link part_5
- removed link part_6
- added link part_7r; visual mesh filename=file:///home/phorce/Desktop/SIGMA/cad/meshes/part_7r.stl scale=0.001 0.001 0.001
- added link part_8r; visual mesh filename=file:///home/phorce/Desktop/SIGMA/cad/meshes/part_8r.stl scale=0.001 0.001 0.001
Joints:
- removed joint fix_part_5
- removed joint fix_part_6
- removed joint fix_part_7
- added joint fix_part_7r: type fixed, parent part_0, child part_7r, origin xyz=0.000000 0.000000 0.000000 rpy=0 0 0
- added joint fix_part_8r: type fixed, parent part_0, child part_8r, origin xyz=0.000000 0.000000 0.000000 rpy=0 0 0
- added joint joint_platform: type revolute, parent part_1, child part_7, origin xyz=-0.006377 -0.029000 0.280777 rpy=0 0 0, axis 0 1 0, limit lower=-1.57 upper=1.57 effort=7.2 velocity=15.7
- joint fix_part_8: parent part_2 -> part_0

Commit message: ADD: Full Sim

File: cad/sigma.urdf (robot description, URDF)
Before this commit: robot sigma, 19 links, 18 joints
Links:
- removed link part_0
- removed link part_1
- removed link part_1r
- removed link part_2
- removed link part_2r
- removed link part_3
- removed link part_3r
- removed link part_4
- removed link part_4r
- removed link part_7
- removed link part_7r
- removed link part_8
- removed link part_8r
- removed link part_9
- added link disc_2; visual mesh filename=file:///home/phorce/Desktop/SIGMA/cad/meshes/disc_2.stl scale=0.001 0.001 0.001
- added link disc_3; visual mesh filename=file:///home/phorce/Desktop/SIGMA/cad/meshes/disc_3.stl scale=0.001 0.001 0.001
- added link lower_0; visual mesh filename=file:///home/phorce/Desktop/SIGMA/cad/meshes/lower_0.stl scale=0.001 0.001 0.001
- added link lower_1; visual mesh filename=file:///home/phorce/Desktop/SIGMA/cad/meshes/lower_1.stl scale=0.001 0.001 0.001
- added link lower_2; visual mesh filename=file:///home/phorce/Desktop/SIGMA/cad/meshes/lower_2.stl scale=0.001 0.001 0.001
- added link lower_3; visual mesh filename=file:///home/phorce/Desktop/SIGMA/cad/meshes/lower_3.stl scale=0.001 0.001 0.001
- added link platform; visual mesh filename=file:///home/phorce/Desktop/SIGMA/cad/meshes/platform.stl scale=0.001 0.001 0.001
- added link upper_0; visual mesh filename=file:///home/phorce/Desktop/SIGMA/cad/meshes/upper_0.stl scale=0.001 0.001 0.001
- added link upper_1; visual mesh filename=file:///home/phorce/Desktop/SIGMA/cad/meshes/upper_1.stl scale=0.001 0.001 0.001
- added link upper_2; visual mesh filename=file:///home/phorce/Desktop/SIGMA/cad/meshes/upper_2.stl scale=0.001 0.001 0.001
- added link upper_3; visual mesh filename=file:///home/phorce/Desktop/SIGMA/cad/meshes/upper_3.stl scale=0.001 0.001 0.001
Joints:
- removed joint fix_part_0
- removed joint fix_part_1
- removed joint fix_part_1r
- removed joint fix_part_2
- removed joint fix_part_2r
- removed joint fix_part_3
- removed joint fix_part_3r
- removed joint fix_part_4
- removed joint fix_part_4r
- removed joint fix_part_7r
- removed joint fix_part_8
- removed joint fix_part_8r
- removed joint fix_part_9
- added joint fix_disc_2: type fixed, parent axis_2, child disc_2, origin xyz=0.000000 0.000000 0.000000 rpy=0 0 0
- added joint fix_disc_3: type fixed, parent axis_3, child disc_3, origin xyz=0.000000 0.000000 0.000000 rpy=0 0 0
- added joint fix_lower_0: type fixed, parent axis_0, child lower_0, origin xyz=0.000000 0.000000 0.000000 rpy=0 0 0
- added joint fix_lower_1: type fixed, parent axis_1, child lower_1, origin xyz=0.000000 0.000000 0.000000 rpy=0 0 0
- added joint fix_lower_2: type fixed, parent axis_2, child lower_2, origin xyz=0.000000 0.000000 0.000000 rpy=0 0 0
- added joint fix_lower_3: type fixed, parent axis_3, child lower_3, origin xyz=0.000000 0.000000 0.000000 rpy=0 0 0
- added joint fix_upper_0: type fixed, parent lower_0, child upper_0, origin xyz=0.000000 0.000000 0.000000 rpy=0 0 0
- added joint fix_upper_1: type fixed, parent lower_1, child upper_1, origin xyz=0.000000 0.000000 0.000000 rpy=0 0 0
- added joint fix_upper_2: type fixed, parent lower_2, child upper_2, origin xyz=0.000000 0.000000 0.000000 rpy=0 0 0
- added joint fix_upper_3: type fixed, parent lower_3, child upper_3, origin xyz=0.000000 0.000000 0.000000 rpy=0 0 0
- joint joint_axis_0: origin xyz=0.060000 0.037000 0.050000 rpy=0 0 0 -> xyz=0.060000 0.107000 0.056000 rpy=0 0 0
- joint joint_axis_1: origin xyz=0.060000 0.113000 0.050000 rpy=0 0 0 -> xyz=0.060000 0.183000 0.056000 rpy=0 0 0
- joint joint_axis_2: origin xyz=0.260000 0.037000 0.050000 rpy=0 0 0 -> xyz=0.260000 0.107000 0.056000 rpy=0 0 0
- joint joint_axis_3: origin xyz=0.260000 0.113000 0.050000 rpy=0 0 0 -> xyz=0.260000 0.183000 0.056000 rpy=0 0 0
- joint joint_platform: child part_7 -> platform; origin xyz=-0.006377 -0.029000 0.280777 rpy=0 0 0 -> xyz=-0.024522 -0.032190 0.226933 rpy=0 0 0; parent part_1 -> upper_0

Commit message: FIX: UDRF

File: cad/sigma.urdf (robot description, URDF)
Before this commit: robot sigma, 16 links, 15 joints
Joints:
- removed joint fix_lower_1
- removed joint fix_lower_2
- removed joint fix_lower_3
- removed joint fix_upper_0
- removed joint fix_upper_1
- removed joint fix_upper_2
- removed joint fix_upper_3
- removed joint joint_axis_1
- removed joint joint_axis_2
- removed joint joint_axis_3
- added joint fix_axis_1: type fixed, parent lower_1, child axis_1, origin xyz=0.111543 -0.032018 -0.103942 rpy=0 0 0
- added joint fix_axis_2: type fixed, parent lower_2, child axis_2, origin xyz=-0.062809 0.032104 -0.138101 rpy=0 0 0
- added joint fix_axis_3: type fixed, parent lower_3, child axis_3, origin xyz=0.088339 -0.032104 -0.123340 rpy=0 0 0
- added joint joint_bearing_1: type revolute, parent platform, child upper_1, origin xyz=0.004001 0.140344 0.000433 rpy=0 0 0, axis 0 1 0, limit lower=-1.57 upper=1.57 effort=7.2 velocity=15.7
- added joint joint_bearing_2: type revolute, parent platform, child upper_2, origin xyz=0.197561 -0.000074 0.033650 rpy=0 0 0, axis 0 1 0, limit lower=-1.57 upper=1.57 effort=7.2 velocity=15.7
- added joint joint_bearing_3: type revolute, parent platform, child upper_3, origin xyz=0.200801 0.140416 0.033996 rpy=0 0 0, axis 0 1 0, limit lower=-1.57 upper=1.57 effort=7.2 velocity=15.7
- added joint joint_knee_0: type revolute, parent lower_0, child upper_0, origin xyz=0.088333 -0.031333 0.124080 rpy=0 0 0, axis 0 1 0, limit lower=-1.57 upper=1.57 effort=7.2 velocity=15.7
- added joint joint_knee_1: type revolute, parent upper_1, child lower_1, origin xyz=-0.091022 -0.000135 -0.123424 rpy=0 0 0, axis 0 1 0, limit lower=-1.57 upper=1.57 effort=7.2 velocity=15.7
- added joint joint_knee_2: type revolute, parent upper_2, child lower_2, origin xyz=0.089769 0.000159 -0.122482 rpy=0 0 0, axis 0 1 0, limit lower=-1.57 upper=1.57 effort=7.2 velocity=15.7
- added joint joint_knee_3: type revolute, parent upper_3, child lower_3, origin xyz=-0.064619 -0.000122 -0.137589 rpy=0 0 0, axis 0 1 0, limit lower=-1.57 upper=1.57 effort=7.2 velocity=15.7
- joint joint_platform: origin xyz=-0.024522 -0.032190 0.226933 rpy=0 0 0 -> xyz=-0.112854 -0.000856 0.102854 rpy=0 0 0
